Commit message: Working urdf model file

File: description/tern/tern.urdf (robot description, URDF)
Before this commit: robot tern, 7 links, 6 joints
Links:
- link left_elevon: mass 0.001 -> 0.02
- link right_elevon: mass 0.001 -> 0.02
- link rotor_left: mass 0.005 -> 0.01; geometry collision box size=0.20 0.02 0.005; visual mesh filename=package://urdf_tutorial/meshes/iris_prop_cw.dae scale=1 1 1
- link rotor_right: mass 0.005 -> 0.01; geometry collision box size=0.20 0.02 0.005; visual mesh filename=package://urdf_tutorial/meshes/iris_prop_ccw.dae scale=1 1 1
Joints:
- joint left_rotor_joint: limit lower=-1000 upper=1000 effort=1.0 velocity=1000.0 -> (none)
- joint right_rotor_joint: limit lower=-1000 upper=1000 effort=1.0 velocity=1000.0 -> (none)
